Commit message: social nav impl, local planner + low-level controller

File: urdf/human_box.urdf.xacro (robot description, xacro)
@@ -5,4 +5,5 @@
   <xacro:arg name="traj_y" default="0.0" />
   <xacro:arg name="traj_z" default="0.0" />
+  <xacro:arg name="enable_motion_plugin" default="true" />
   <material name="human_blue">
     <color rgba="0.0 0.4 0.8 1"/>
@@ -15,5 +16,5 @@
     </inertial>
     <visual>
-        <origin xyz="0 0 0.9" rpy="0 0 0" />
+        <origin xyz="-10.0 -10.0 0.9" rpy="0 0 0" />
         <geometry>
           <box size="0.6 0.8 1.8"/>
@@ -22,5 +23,5 @@
     </visual>
     <collision>
-        <origin xyz="0 0 0.9" rpy="0 0 0" />
+        <origin xyz="-10.0 -10.0 0.9" rpy="0 0 0" />
         <geometry>
           <box size="0.6 0.8 1.8"/>
@@ -32,10 +33,12 @@
     <material>Gazebo/Blue</material>
   </gazebo>
-  <gazebo>
-    <plugin name="move_model" filename="libmove_model.so">
-      <traj_x>$(arg traj_x)</traj_x>
-      <traj_y>$(arg traj_y)</traj_y>
-      <traj_z>$(arg traj_z)</traj_z>
-    </plugin>
-  </gazebo>
+  <xacro:if value="$(arg enable_motion_plugin)">
+    <gazebo>
+      <plugin name="move_model" filename="libmove_model.so">
+        <traj_x>$(arg traj_x)</traj_x>
+        <traj_y>$(arg traj_y)</traj_y>
+        <traj_z>$(arg traj_z)</traj_z>
+      </plugin>
+    </gazebo>
+  </xacro:if>
 </robot>

File: urdf/p3at.urdf.xacro (robot description, xacro)
@@ -22,5 +22,5 @@
   <!-- <xacro:p3at_gazebo_ext name="$(arg namespace)_red_rover" namespace="$(arg namespace)" /> -->
   <xacro:include filename="$(find ros2_livox_simulation)/urdf/mid360.xacro" />
-  <xacro:mid360 name="$(arg namespace)_livox" namespace="$(arg namespace)" parent="base_link" topic="mid360" lidar_update_rate="10" >
+  <xacro:mid360 name="$(arg namespace)_livox" namespace="$(arg namespace)" parent="base_link" topic="mid360" >
     <origin xyz="0 0 1.0" rpy="0 0.3 0"/>
   </xacro:mid360>
